File: PCB_Files/TickerPCB.kicad_sch (KiCad schematic)
At the start: 105 parts

Commit message: Clean up schematic
Parts:
- B0, B1, B2, B3, B4, B5, B6, B7: value (none) -> Button
- B8: value (none) -> MAX17623
- C1, C10, C7, C8, C9: value (none) -> 10uF
- C11, C13, C3, C30, C5: value (none) -> 1uF
- C12: value (none) -> 100nF 0603
- C14: value (none) -> 47uF 0805
- C15: value (none) -> 22pF 0603
- C16, C17, C18, C19, C20, C21, C22, C23, C24, C25: value (none) -> 0.1uF 0603
- C2, C26: value (none) -> 2.2uF
- C4: value (none) -> 0.1uF
- C6: value (none) -> 100uF
- D1: value (none) -> LTST-C170TBKT
- D2: value (none) -> HSMS-C170
- DS1, DS3: value (none) -> HSMG-C170
- DS2: value (none) -> HSMD-C170
- ESP1: value (none) -> ESP8266
- H0, H1, H2, H3: value (none) -> LiteOn14Seg
- J1: value (none) -> 105017-0001
- L1: value (none) -> 6.8uH
- L2: value (none) -> 1uH
- M1: value (none) -> MAX6955
- M2: value (none) -> SI1499dh
- MC1: value (none) -> MCP73871
- P1: value (none) -> S2B-PH-SM4-TB(LF)(SN)
- P2: value (none) -> PDTA143Z
- R1, R3: value (none) -> 1.87M
- R10, R19, R6, R9: value (none) -> 4.7k
- R11: value (none) -> 56k
- R12: value (none) -> 300
- R13, R4: value (none) -> 200k
- R14, R8: value (none) -> 470
- R15, R18, R21, R22, R23, R24, R25, R26, R29: value (none) -> 10k
- R16: value (none) -> 1k
- R17, R7: value (none) -> 100k
- R2: value (none) -> 340k
- R20, R27, R28, R5: value (none) -> 200
- R30: value (none) -> 118k
- R31: value (none) -> 37.4k
- R32: value (none) -> 3.9k
- R33: value (none) -> 6.34k
- R6: value (none) -> 270k
- SW1: value (none) -> JS202011SCQN
- T1: value (none) -> TPS61090
- THERM: value (none) -> 16k
- U1: value (none) -> 3.3V-5V Level Shifter
- U10, U11, U12, U13, U14, U5, U6, U7, U8, U9: value (none) -> NeoPixel1655
- U19: value (none) -> TCA9534PWR
- U2, U4: value (none) -> MCP9808-E/MS
Other:
- note added: "14-Segment Display Driver (I2C)"
- note added: "14-Segment Displays"
- note added: "3.3V - 5V Level Shifter"
- note added: "Battery Charge Management Controller"
- note added: "Battery connector"
- note added: "Battery level indication LEDs"
- note added: "Boost Converter: VBAT to 5V"
- note added: "Buck Converter: VBAT to 3.3V"
- note added: "Buttons"
- note added: "ESP8266 Microcontroller Board"
- note added: "GPIO Expander (I2C)"
- note added: "NeoPixel LEDS"
- note added: "Switch to connect BMS output to OUT Voltage or GND"
- note added: "Temperature Sensors (I2C)"
- note added: "This mosfet allows VCC(3.3V) to power the ESP8622's 3.3V pins when powered from the battery. When the ESP8622 is powered from the dev board, ESPVIN(5V) will turn off this P-Channel Mosfet and therefore leave VCC disconnnected, so only the dev board will be powered."
- note added: "USB 5V input"
- note added: "USB Power Connector"
- note added: "Voltage Direction Protection"
- moved on the sheet: B0, B1, B2, B3, B4, B5, B6, B7, B8, C1, C10, C11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

Commit message: finish cleaning up schematic
Parts:
- C12: value 100nF 0603 -> 100nF
- C14: value 47uF 0805 -> 47uF
Other:
- note added: "ESP8266 Microcontroller Dev Board"
- note added: "I2C Sensors & Controllers"
- note added: "Inputs"
- note added: "MCU"
- note added: "Outputs"
- note added: "PCB Interfacing"
- note added: "Power"
- note removed: "ESP8266 Microcontroller Board"
- note removed: "Power Section"
- moved on the sheet: B0, B1, B2, B3, B4, B5, B6, B7, B8, C1, C10, C11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
